File: radio/radio.kicad_sch (KiCad schematic)
At the start: 0 parts

Commit message: wee
Parts:
- added AE1: Antenna, footprints:ANT_GP.1575.18.4.A.02_TAL, symbol Device:Antenna
- added BT1: Battery, Connector_JST:JST_XH_S2B-XH-A_1x02_P2.50mm_Horizontal, symbol Device:Battery
- added C1: 0.1uf, Capacitor_SMD:C_1812_4532Metric, symbol Device:C
- added C2, C3, C4, C5, C6: 1uF, Capacitor_SMD:C_1206_3216Metric, symbol Device:C
- added C7, C8: 2.2uF, Capacitor_SMD:C_1206_3216Metric, symbol Device:C
- added C9: 2.2 uF, Capacitor_SMD:C_1206_3216Metric, symbol Device:C
- added D1, D2: LED, LED_SMD:LED_01005_0402Metric_Pad0.57x0.30mm_HandSolder, symbol Device:LED
- added J1: Conn_Coaxial_Small, Connector_Coaxial:SMA_Amphenol_132291_Vertical, symbol Connector:Conn_Coaxial_Small
- added P1: USB_C_Plug_USB2.0, Connector_USB:USB_C_Receptacle_Amphenol_124019772112A, symbol Connector:USB_C_Plug_USB2.0
- added R1: 5.1k, Resistor_SMD:R_1225_3264Metric, symbol Device:R
- added R2: 100, Resistor_SMD:R_1225_3264Metric, symbol Device:R
- added R3: 200, Resistor_SMD:R_1225_3264Metric, symbol Device:R
- added SW1, SW2, SW3, SW4: SW_Push, Button_Switch_SMD:SW_Push_SPST_NO_Alps_SKRK, symbol Switch:SW_Push
- added U1: MCP2221AxML, Package_DFN_QFN:QFN-16-1EP_4x4mm_P0.65mm_EP2.5x2.5mm, symbol Interface_USB:MCP2221AxML
- added U2: RAK811-HF-US915, RF_Module:RAK811, symbol RF_Module:RAK811-HF-US915
- added U3: BQ24013, Package_SON:Texas_DRC0010J_ThermalVias, symbol Battery_Management:BQ24013
- added U4: NHD-C12832A1Z-FSRGB, Display:NHD-C12832A1Z-FSRGB, symbol Display_Graphic:NHD-C12832A1Z-FSRGB
- added U6: MIA-M10Q, Package_LGA:ublox_LGA-53_4.5x4.5mm_Layout9x9_P0.5mm, symbol RF_GPS:MIA-M10Q
Connections:
- new net: SW4.2, U4.16 (~{RST})
- new net: D2.2 (A), U3.4 (STAT2)
- new net: C6.1, U4.5 (V4)
- new net: D1.2 (A), U3.3 (STAT1)
- new net: SW3.1, U2.17 (BOOT0)
- new net: SW2.2, U2.24 (~{RST})
- new net: J1.1 (In), U2.33 (RF_OUT)
- new net: U1.4 (URx), U2.6 (PA9/USART1_TX)
- new net: U1.5 (UTx), U2.7 (PA10/USART1_RX)
- new net: C2.2, U4.1 (V0)
- new net: C7.1, U4.10 (V_{out})
- new net: C3.1, U4.2 (V1)
- new net: C4.2, U4.3 (V2)
- new net: C5.2, U4.4 (V3)
- new net: C9.2, U4.6 (C2-)
- new net: C9.1, U4.7 (C2+)
- new net: C8.1, U4.8 (C1+)
- new net: C8.2, U4.9 (C1-)
- new net: AE1.1 (A), U6.B9 (RF_IN)
- new net: P1.A5 (CC), R1.2
- new net: SW1.2, U1.3 (~{RST})
- new net: C1.2, U3.6 (ISET)
- new net +3.3V: BT1.1 (+), C1.1, SW1.1, SW2.1, SW3.2, U1.10 (VUSB), U1.16 (VDD), U2.11 (VCC), U3.10 (OUT), U3.9 (BAT), U4.12 (V_{dd}), U6.B1 (VCC), U6.C6 (VCC_RF), U6.H9 (LNA_EN), U6.J4 (V_IO)
- new net +3.3V USB: P1.B5 (VCONN), R2.2, R3.1, U3.1 (IN), U3.2 (VCC)
- new net +3V0: SW4.1
- new net +5V: P1.A4 (VBUS), P1.A9 (VBUS), P1.B4 (VBUS), P1.B9 (VBUS), R2.1
- new net A0: U2.9 (PB4), U4.15 (A0)
- new net GND: BT1.2 (-), C2.1, C3.2, C4.1, C5.1, C6.2, C7.2, D1.1 (K), D2.1 (K), J1.2 (Ext), P1.A1 (GND), P1.A12 (GND), P1.B1 (GND), P1.B12 (GND), P1.SH (SHIELD), R1.1, R3.2, U1.13 (VSS), U2.1 (GND), U2.12 (GND), U2.21 (GND), U2.28 (GND), U2.29 (GND), U2.30 (GND), U2.31 (GND), U2.32 (GND), U2.34 (GND), U3.11 (VSS), U3.5 (VSS), U3.7 (~{CE}), U3.8 (~{TTE}), U4.11 (V_{ss}), U4.17 (~{CS1B}), U4.19 ((R)LED-), U4.20 ((G)LED-), U4.21 ((B)LED-), U6.A1 (GND), U6.A2 (GND), U6.A3 (GND), U6.A5 (RTC_O), U6.A8 (GND), U6.A9 (GND), U6.B2 (GND), U6.B8 (GND), U6.C3 (GND), U6.C9 (GND), U6.E3 (GND), U6.E4 (GND), U6.E9 (GND), U6.F1 (GND), U6.F3 (GND), U6.F4 (GND), U6.G3 (GND), U6.G4 (GND), U6.G5 (GND), U6.G6 (GND), U6.H8 (GND), U6.J8 (GND), U6.J9 (GND)
- new net GPS_Boot: U6.C7 (~{SAFEBOOT})
- new net GPS_RST: U6.C4 (~{RESET})
- new net SCL: U2.18 (PB8), U4.14 (SCL)
- new net SDA: U2.19 (PB9), U4.13 (SDA(SI))
- new net d_minus: P1.A7 (D-), U1.11 (D-)
- new net d_plus: P1.A6 (D+), U1.12 (D+)
- no-connect marks 0 -> 15
